File: mech/kicad/hawkeye_driver/hawkeye_driver.kicad_pcb (KiCad board)
At the start: 2 copper layers, 71.1 x 54.6 mm, 31 parts, among them J1 Conn_01x03_Male, J2 Screw_Terminal_01x02, Q1 IRLD024, Q2 IRLD024, Q3 IRLD024, U1 74HC595

Commit message: work on ground planes
Parts:
- removed R20: 2k, Resistor_THT:R_Axial_DIN0207_L6.3mm_D2.5mm_P5.08mm_Vertical
- removed R21: 5k, Resistor_THT:R_Axial_DIN0207_L6.3mm_D2.5mm_P5.08mm_Vertical
- added C1: 1 uF, Capacitor_SMD:C_1206_3216Metric_Pad1.33x1.80mm_HandSolder, F.Cu at (112.4, 79.4)
- J1: value Conn_01x03_Male -> Conn_02x05_Odd_Even; footprint Connector_PinHeader_2.54mm:PinHeader_1x03_P2.54mm_Vertical -> Connector_IDC:IDC-Header_2x05_P2.54mm_Vertical
- R14, R15, R16, R17, R18, R19: footprint Resistor_THT:R_Axial_DIN0207_L6.3mm_D2.5mm_P5.08mm_Vertical -> Resistor_SMD:R_1206_3216Metric_Pad1.30x1.75mm_HandSolder
- moved R14 17.8 mm to (167.6, 106.7)
- moved R19 16.1 mm to (167.6, 88.9), turned to -90 degrees
- moved Q1 12.7 mm to (162.6, 104.1), turned to -90 degrees
- moved Q3 12.7 mm to (162.6, 91.4), turned to -90 degrees
- moved R17 9.16 mm to (167.6, 101.6), turned to -90 degrees
- moved R18 9.16 mm to (167.6, 76.2), turned to -90 degrees
- moved J1 8.35 mm to (118.7, 113.0), turned to 90 degrees
- moved R16 5.08 mm to (167.6, 94.0)
- moved R15 2.54 mm to (167.6, 81.3)
- turned Q2 to -90 degrees
Connections:
- J1 pad 1: /SHIFT CLK -> GND
- J1 pad 2: /LATCH -> /5V
- J1 pad 3: /SER IN -> GND
- U1 pad 10: /4.78 V (req. > 4V) -> /5V
- U1 pad 16: /4.78 V (req. > 4V) -> /5V
Routing:
- net VCC: track 145.4 -> 0.00 mm
- net Net-(Q2-Pad1): track 111.2 -> 0.00 mm
- net Net-(R17-Pad1): track 90.8 -> 0.00 mm, vias 1 -> 0
- net Net-(Q1-Pad1): track 81.8 -> 0.00 mm
- net Net-(R19-Pad1): track 80.6 -> 0.00 mm, vias 1 -> 0
- net Net-(R18-Pad1): track 79.3 -> 0.00 mm, vias 1 -> 0
- net /SHIFT CLK: track 35.0 -> 0.00 mm
- net Net-(Q3-Pad1): track 34.3 -> 0.00 mm
- net /LATCH: track 30.8 -> 0.00 mm
- net /4.78 V (req. > 4V): track 25.9 -> 0.00 mm
- net /SER IN: track 25.3 -> 0.00 mm
- net Net-(Q2-Pad2): track 11.3 -> 9.83 mm
- net Net-(Q3-Pad2): track 9.09 -> 9.83 mm
- added copper zone on B.Cu, net Net-(Q2-Pad1)
- added copper zone on B.Cu, net Net-(Q3-Pad1)
- added copper zone on F.Cu, net VCC
- removed copper zone on F.Cu, net GND

Commit message: finish ground plane rework
Parts:
- C1: value 1 uF -> .1 uF
- R14, R15, R16, R17, R18, R19: moved to B.Cu
- moved C1 13.9 mm to (119.4, 91.4), turned to 90 degrees
- moved R14 2.54 mm to (170.2, 106.7)
- moved R15 2.54 mm to (170.2, 81.3)
- moved R16 2.54 mm to (170.2, 94.0)
- moved R17 2.54 mm to (170.2, 101.6)
- moved R18 2.54 mm to (170.2, 76.2)
- moved R19 2.54 mm to (170.2, 88.9)
- moved U1 1.91 mm to (112.4, 91.4), turned to -90 degrees
Connections:
- net Net-(Q1-Pad1) renamed /INNER_RING_LOW
- net Net-(Q2-Pad1) renamed /OUTER_RING_LOW
- net Net-(Q3-Pad1) renamed /CENTER_LOW
- C1 pad 2: GND -> GND1
- J1 pad 1: GND -> GND1
- J1 pad 10: GND -> GND1
- J1 pad 3: GND -> GND1
- J1 pad 4: /SER IN -> /SHIFT CLK
- J1 pad 5: GND -> GND1
- J1 pad 6: /SHIFT CLK -> /LATCH
- J1 pad 7: GND -> GND1
- J1 pad 8: /LATCH -> /SER IN
- J1 pad 9: GND -> GND1
- U1 pad 13: GND -> GND1
- U1 pad 8: GND -> GND1
Routing:
- net Net-(R19-Pad1): track 0.00 -> 97.0 mm, vias 0 -> 3
- net Net-(R17-Pad1): track 0.00 -> 89.6 mm, vias 0 -> 1
- net Net-(R18-Pad1): track 0.00 -> 70.0 mm, vias 0 -> 1
- net GND1: track 0.00 -> 57.6 mm, vias 0 -> 3
- net /5V: track 0.28 -> 31.9 mm, vias 0 -> 2
- net /SER IN: track 0.00 -> 23.7 mm
- net /LATCH: track 0.00 -> 22.6 mm
- net /SHIFT CLK: track 0.00 -> 20.9 mm
- net GND: track 0.00 -> 19.7 mm
- net Net-(Q3-Pad2): track 9.83 -> 12.4 mm
- net Net-(Q2-Pad2): track 9.83 -> 12.4 mm
- net Net-(Q1-Pad2): track 9.83 -> 12.4 mm
- added copper zone on B.Cu, net /INNER_RING_LOW
- added copper zone on F.Cu, net GND
Other:
- board text added: "5V"
- board text added: "PICO"
- board text added: "SCK"
- board text removed: "CLK"
- board text removed: "SER_IN"
