File: mech/kicad/hawkeye_driver/hawkeye_driver.kicad_pcb (KiCad board)
At the start: 2 copper layers, 71.1 x 54.6 mm, 30 parts, among them J1 Conn_02x05_Odd_Even, J2 Screw_Terminal_01x02, Q1 IRLD024, Q2 IRLD024, Q3 IRLD024, U1 74HC595

Commit message: final commit before fab
Connections:
- J1 pad 10: GND1 -> unconnected-(J1-Pad10)
Routing:
- net GND1: track 57.6 -> 16.8 mm, vias 3 -> 2
- added copper zone on B.Cu, net GND1
Other:
- board text added: "."
